File: KiCad/JSB01.kicad_sch (KiCad schematic)
At the start: 25 parts, among them J1 MB10XX Sonar, J2 VL53LXX TOF(0x29), M1 LD14, Q2 AO3400A, SW1 Tactile, SW2 Tactile, SW3 Slide, U1 TPS61291DRVR, U2 QMC5883L(0x0D), U3 BH1750FVI(0x23)

Commit message: BTO ver. (QMC5883P)
Parts:
- removed BT1: 2xAAA, JSB01_Lib:BatteryHolder 2xAAA, symbol Device:Battery
- removed C3: 0.22uF, Capacitor_SMD:C_0603_1608Metric, symbol Device:C
- removed J2: VL53LXX TOF(0x29), Connector_PinSocket_2.54mm:PinSocket_1x06_P2.54mm_Vertical, symbol Connector:Conn_01x06_Socket
- removed MCU1: XIAO RP2040, JSB01_Lib:MOUDLE14P-2.54-21X17.8MM, symbol JSB01_Lib:XIAO RP2040
- removed U1: TPS61291DRVR, JSB01_Lib:WSON-6_L2.0-W2.0-P0.65-BL-EP, symbol JSB01_Lib:TPS61291DRVR
- removed U2: QMC5883L(0x0D), JSB01_Lib:LGA-16_L3.0-W3.0-P0.50-BL_SQ, symbol JSB01_Lib:QMC5883L
- added BT1: 1xAAA, JSB01_Lib:BatteryHolder_SN4_1PC, symbol Device:Battery_Cell
- added C10, C9: 33p, Capacitor_SMD:C_0603_1608Metric, symbol Device:C
- added C11, C12, C13, C14, C15, C16, C17, C18, C19, C20: 100n, Capacitor_SMD:C_0402_1005Metric, symbol JSB01_Lib:Bypass_C
- added C21: 100u, JSB01_Lib:CAP-SMD_L6.0-W3.2, symbol Device:C_Polarized_US
- added C7, C8: 10u, Capacitor_SMD:C_0603_1608Metric, symbol Device:C
- added D1: LED, JSB01_Lib:LED0603-RD_GREEN, symbol JSB01_Lib:LED_Green
- added D2: NSR0320MW2T1G, JSB01_Lib:SOD-323_L1.8-W1.3-LS2.5-RD, symbol JSB01_Lib:Schottky_Diode
- added D3: 1N5819WS, JSB01_Lib:SOD-323_L1.8-W1.3-LS2.5-RD, symbol JSB01_Lib:Schottky_Diode
- added J2: USB_C_Receptacle_USB2.0, JSB01_Lib:USB-C-SMD_TYPE-C-16P-1, symbol JSB01_Lib:USB_C_Receptacle_USB2.0
- added JP2: SolderJumper_2_Open, Jumper:SolderJumper-2_P1.3mm_Open_RoundedPad1.0x1.5mm, symbol JSB01_Lib:SolderJumper_2_Bridged
- added JP3: SolderJumper_2_Open, JSB01_Lib:SolderJumper-2_Open_mini, symbol Jumper:SolderJumper_2_Open
- added R10, R11: 27.4, Resistor_SMD:R_0402_1005Metric, symbol Device:R
- added R12: 470, Resistor_SMD:R_0603_1608Metric, symbol Device:R
- added R13: 470K, Resistor_SMD:R_0603_1608Metric, symbol Device:R
- added R14: 390K, Resistor_SMD:R_0603_1608Metric, symbol Device:R
- added R15: 1M, Resistor_SMD:R_0603_1608Metric, symbol Device:R
- added R3, R4: 5.1K, Resistor_SMD:R_0402_1005Metric, symbol Device:R
- added R8: 1K, Resistor_SMD:R_0603_1608Metric, symbol Device:R
- added R9: 1k, Resistor_SMD:R_0603_1608Metric, symbol Device:R
- added SW4, SW5: SKRPABE010, JSB01_Lib:KEY-SMD_4P-L4.2-W3.2, symbol JSB01_Lib:Button_SMD
- added U1: RP2040, JSB01_Lib:RP2040-QFN-56, symbol JSB01_Lib:RP2040
- added U2: W25Q128JVSIQ, JSB01_Lib:SOP-8-208mil, symbol JSB01_Lib:W25Q128JVSIQ
- added U3: TPS61025DRCR, JSB01_Lib:VSON-10_L3.0-W3.0-P0.50-BL-EP, symbol JSB01_Lib:TPS61025DRCR
- added U4: AMS1117-3.3, JSB01_Lib:SOT-223-3_L6.5-W3.4, symbol JSB01_Lib:AMS1117-3.3
- added U5: QMC5883P(0x2C), JSB01_Lib:LGA-16_L3.0-W3.0-P0.50-BL_SQ, symbol JSB01_Lib:QMC5883P
- added Y1: TAXM12M4RLBDDT2T, JSB01_Lib:OSC-SMD_4P-L3.2-W2.5, symbol JSB01_Lib:Crystal_GND24
- C1: value 10uF -> 10u
- C2: value 22uF -> 2.2u; LCSC C59461 -> C23630
- C4: value 0.1uF -> 0.1u
- C5: value 4.7uF -> 4.7u
- C6: value 1uF -> 1u
- L1: value 3.3μH -> 6.8μH; LCSC C136236 -> C404497
- Q2: footprint Package_TO_SOT_SMD:SOT-23 -> JSB01_Lib:AO3400A
- R1, R2: value 10KΩ -> 4.7K; LCSC C25804 -> C23162
- R5: value 100KΩ -> 100K
- R6: value 20KΩ -> 20K
- SW1, SW2: footprint JSB01_Lib:SW_tactile_DTS6 -> JSB01_Lib:SW-SMD_4P-L4.5-W4.5-P3.00-LS6.8; symbol Switch:SW_Push -> JSB01_Lib:SW_Tactile4P; LCSC (none) -> C2888900; now in the parts list
- renumbered U3 to U6
Connections:
- net GND: now also SW1.3, SW1.4, SW2.3, SW2.4, U6.7 (EP), BT1.2 (-), C10.1, C11.2, C12.2, C13.2, C14.2, C15.2, C16.2, C17.2, C18.2, C19.2, C20.2, C21.2, C7.2, C8.2, C9.1, D1.1 (K), J2.A1B12 (GND), J2.B1A12 (GND), J2.EP, R14.2, R3.2, R4.2, SW4.1, SW5.1, U1.19 (TESTEN), U1.57 (GND), U2.4 (GND), U3.10 (PGND), U3.11 (EP), U3.5 (GND), U3.8 (PS), U4.1 (GND), U5.11 (GND), U5.9 (GND), Y1.2 (GND), Y1.4 (GND); no longer SW1.2, SW2.2
- net SCL: now reaches R2.2, U6.6 (SCL)
- net SCL: now also U1.7 (GPIO5), U5.1 (SCL)
- net SONAR_PW: now reaches J1.6 (PW)
- net SONAR_PW: now also U1.8 (GPIO6)
- net SDA: now reaches R1.2, U6.4 (SDA)
- net SDA: now also U1.6 (GPIO4), U5.16 (SDA)
- net at C1.1, JP1.1 (A), L1.1: now also JP2.2 (B), JP3.1 (A), R13.1, U3.1 (EN), U3.6 (VBAT)
- net at L1.2: now also U3.9 (SW)
- net at C5.1: now also U5.10 (C1)
- net SW1: now reaches SW1.1
- net SW1: now also SW1.2, U1.2 (GPIO0)
- net SW2: now reaches SW2.1
- net SW2: now also SW2.2, U1.3 (GPIO1)
- net VIB: now reaches R6.1
- net VIB: now also U1.4 (GPIO2)
- net at JP1.2 (C), SW3.1 (A): now also JP2.1 (A)
- net at SW3.2 (B): now also BT1.1 (+)
- net +3.3V renamed +3V3
- net +3V3: now also C11.1, C12.1, C14.1, C16.1, C18.1, C19.1, C20.1, C21.1, D3.1 (K), R15.2, U1.1 (IOVDD), U1.10 (IOVDD), U1.22 (IOVDD), U1.33 (IOVDD), U1.42 (IOVDD), U1.43 (ADC_AVDD), U1.44 (VREG_IN), U1.48 (USB_VDD), U1.49 (IOVDD), U2.8 (VCC), U3.2 (VOUT), U5.2 (VDD)
- new net: C8.1, D3.2 (A), U4.2 (VOUT), U4.4 (VOUT)
- new net: R9.1, SW4.2
- new net: C7.1, D2.1 (K), U4.3 (VIN)
- new net: D2.2 (A), J2.A4B9 (VBUS), J2.B4A9 (VBUS)
- new net: C10.2, R8.1, Y1.3 (OSC2)
- new net: D1.2 (A), R12.1
- new net: J2.B5 (CC2), R3.1
- new net: J2.A5 (CC1), R4.1
- new net: R13.2, R14.1, U3.7 (LBI)
- new net: R10.2, U1.47 (USB_DP)
- new net: R12.2, U1.37 (GPIO25)
- new net: R11.2, U1.46 (USB_DM)
- new net +1V1: C13.1, C15.1, C17.1, U1.23 (DVDD), U1.45 (VREG_VOUT), U1.50 (DVDD)
- new net LBO: R15.1, U1.9 (GPIO7), U3.4 (LBO)
- new net QSPI_SCLK: U1.52 (QSPI_SCLK), U2.6 (CLK)
- new net QSPI_SD0: U1.53 (QSPI_SD0), U2.5 (IO0)
- new net QSPI_SD1: U1.55 (QSPI_SD1), U2.2 (IO1)
- new net QSPI_SD2: U1.54 (QSPI_SD2), U2.3 (IO2)
- new net QSPI_SD3: U1.51 (QSPI_SD3), U2.7 (IO3)
- new net QSPI_SS: R9.2, U1.56 (QSPI_SS), U2.1 (~{CS})
- new net RESET: SW5.2, U1.26 (RUN)
- new net USB_DM: J2.A7 (D-), J2.B7 (D-), R11.1
- new net USB_DP: J2.A6 (D+), J2.B6 (D+), R10.1
- new net VBAT: JP3.2 (B), U1.41 (GPIO29_ADC3)
- new net XIN: C9.2, U1.20 (XIN), Y1.1 (OSC1)
- new net XOUT: R8.2, U1.21 (XOUT)
- no-connect marks 0 -> 28
Other:
- moved on the sheet: C1, C4, C5, C6, J1, JP1, L1, M1, Q2, R1, R2, R5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
